Commit message: Shelf and collisions
Added a shelf to the world and adjusted collisions, inertias and masses

File: dsrbot_description/urdf/DSRbot_URDF.xacro (robot description, xacro)
@@ -1,4 +1,4 @@
 <?xml version="1.0"?>
-<robot name="DSRbot" xmlns:xacro="http://ros.org/wiki/xacro">
+<robot name="DSRbot" xmlns:xacro="http://www.ros.org/wiki/xacro">
 <xacro:include filename="$(find dsrbot_description)/urdf/DSRbot.gazebo" />
   <link name="placeholder_base"/>
@@ -14,12 +14,12 @@
 		</visual>
 		<collision>
-		      <origin xyz="0 0 0" rpy="0 0 0"/>
+		      <origin xyz="1.765 0 0" rpy="0 0 0"/>
 		      <geometry>
-			<box size="3.53 0.3 2"/>
+			<box size="3.53 0.1 2"/>
 		      </geometry>
 		    </collision>
 		        <inertial>
-			      <origin xyz="0 0 0.015" rpy="0 0 0"/>
-			      <mass value="1"/>
+			      <origin xyz="1.765 0 0" rpy="0 0 0"/>
+			      <mass value="2"/>
 			      <inertia ixx="1" ixy="0" ixz="0"
 				       iyy="1" iyz="0"
@@ -44,5 +44,5 @@
 		    </collision>
 		        <inertial>
-			      <origin xyz="0 0 0.015" rpy="0 0 0"/>
+			      <origin xyz="0.075 0.05 0.33" rpy="0 0 0"/>
 			      <mass value="0.1"/>
 			      <inertia ixx="1" ixy="0" ixz="0"
@@ -62,5 +62,5 @@
 		</visual>
 						<collision>
-		      <origin xyz="0 0 0" rpy="0 0 0"/>
+		      <origin xyz="1.7575 0 0.14" rpy="0 0 0"/>
 		      <geometry>
 			<box size="3.5 0.03 0.03"/>
@@ -68,5 +68,5 @@
 		    </collision>
 		        <inertial>
-			      <origin xyz="0 0 0.015" rpy="0 0 0"/>
+			      <origin xyz="1.7575 0 0.14" rpy="0 0 0"/>
 			      <mass value="1"/>
 			      <inertia ixx="1.4e-03" ixy="0" ixz="0"
@@ -85,12 +85,12 @@
 	     		</material>
 		</visual>
-								<collision>
-		      <origin xyz="0 0 0" rpy="0 0 0"/>
-		      <geometry>
+		<collision>
+		    <origin xyz="1.75 0 0" rpy="0 0 0"/>
+		    <geometry>
 			<box size="0.25 0.05 0.33"/>
-		      </geometry>
-		    </collision>
+		    </geometry>
+	    </collision>
 		        <inertial>
-			      <origin xyz="0 0 0.015" rpy="0 0 0"/>
+			      <origin xyz="1.75 0 0" rpy="0 0 0"/>
 			      <mass value="0.1"/>
 			      <inertia ixx="1.4e-03" ixy="0" ixz="0"
@@ -109,5 +109,5 @@
     <child link="soporte1_link"/>
     <axis xyz="0 0 1"/>
-    <limit upper="0.95" lower="-0.83" velocity="10" effort="100"/>
+    <limit upper="0.95" lower="-0.83" velocity="1" effort="100"/>
   </joint>
 <joint name="riel1_joint" type="fixed">

Commit message: Carrier Mesh
Added an STL mesh for the carrier and changed its color

File: dsrbot_description/urdf/DSRbot_URDF.xacro (robot description, xacro)
@@ -77,11 +77,8 @@
    <link name="carrier_link">
 		<visual>
-		    <origin xyz="1.75 0 0" rpy="0 0 0"/>
+		    <origin xyz="1.75 0.1 0.75" rpy="1.5708 0 0"/>
 			<geometry>
-				<box size="0.25 0.05 0.33"/>
+                <mesh filename="$(find dsrbot_description)/meshes/carrier_assy.STL" scale="0.001 0.001 0.001"/>
 			</geometry>
-			<material name="n3">
-	       			<color rgba="1 1 1 1.0"/>
-	     		</material>
 		</visual>
 		<collision>

Commit message: Incorrect positions
The visuals were positioned incorrectly

File: dsrbot_description/urdf/DSRbot_URDF.xacro (robot description, xacro)
@@ -77,5 +77,5 @@
    <link name="carrier_link">
 		<visual>
-		    <origin xyz="1.75 0.1 0.75" rpy="1.5708 0 0"/>
+		    <origin xyz="1.5975 0.1 0.7485" rpy="1.5708 0 0"/>
 			<geometry>
                 <mesh filename="$(find dsrbot_description)/meshes/carrier_assy.STL" scale="0.001 0.001 0.001"/>

Commit message: Position adjustment
Adjusted positions. No position or collision box is exact because i had to rotate the thing 90° and Gazebo does not let me measure things like I'd like.

File: dsrbot_description/urdf/DSRbot_URDF.xacro (robot description, xacro)
@@ -5,11 +5,8 @@
   <link name="base1_link">
 		<visual>
-		    <origin xyz="0 0 0" rpy="0 0 0"/>
+		    <origin xyz="0.04 0.1 1" rpy="1.5708 0 0"/>
 			<geometry>
-				<box size="0.03 0.03 2"/>
+				<mesh filename="$(find dsrbot_description)/meshes/rieles_verticales.STL" scale="0.001 0.001 0.001"/>
 			</geometry>
-			<material name="cyan3">
-	       			<color rgba="0 0.2 0.2 1.0"/>
-	     		</material>
 		</visual>
 		<collision>
@@ -29,20 +26,17 @@
   <link name="soporte1_link">
 		<visual>
-		    <origin xyz="0.0125 0 0" rpy="0 0 0"/>
+		    <origin xyz="0.04 0.1 1.78175" rpy="1.5708 0 0"/>
 			<geometry>
-				<box size="0.075 0.05 0.33"/>
+				<mesh filename="$(find dsrbot_description)/meshes/soportes_verticales.STL" scale="0.001 0.001 0.001"/>
 			</geometry>
-			<material name="cyan2">
-	       			<color rgba="0 0.2 0.2 1.0"/>
-	     		</material>
 		</visual>
-				<collision>
-		      <origin xyz="0 0 0" rpy="0 0 0"/>
+		<collision>
+		    <origin xyz="0.01045 0 0" rpy="0 0 0"/>
 		      <geometry>
 			<box size="0.075 0.05 0.33"/>
 		      </geometry>
-		    </collision>
+        </collision>
 		        <inertial>
-			      <origin xyz="0.075 0.05 0.33" rpy="0 0 0"/>
+			      <origin xyz="0.01045 0 0" rpy="0 0 0"/>
 			      <mass value="0.1"/>
 			      <inertia ixx="1" ixy="0" ixz="0"

Commit message: Mesh implementation
All links have now STL visuals

File: dsrbot_description/urdf/DSRbot_URDF.xacro (robot description, xacro)
@@ -47,11 +47,8 @@
    <link name="riel1_link">
 		<visual>
-		    <origin xyz="1.7575 0 0.14" rpy="0 0 0"/>
+		    <origin xyz="0.045 0.9412 0.015" rpy="0 0 0"/>
 			<geometry>
-				<box size="3.5 0.03 0.03"/>
+				<mesh filename="$(find dsrbot_description)/meshes/rieles_horizontales.STL" scale="0.001 0.001 0.001"/>
 			</geometry>
-			<material name="cyan3">
-	       			<color rgba="0 0.2 0.2 1.0"/>
-	     		</material>
 		</visual>
 						<collision>

Commit message: Tried to correct something but in the end i did nothing
I lost my time

File: dsrbot_description/urdf/DSRbot_URDF.xacro (robot description, xacro)
@@ -5,5 +5,5 @@
   <link name="base1_link">
 		<visual>
-		    <origin xyz="0.04 0.1 1" rpy="1.5708 0 0"/>
+		    <origin xyz="0.04 0.1 0.945" rpy="1.5708 0 0"/>
 			<geometry>
 				<mesh filename="$(find dsrbot_description)/meshes/rieles_verticales.STL" scale="0.001 0.001 0.001"/>
@@ -97,5 +97,5 @@
     <child link="soporte1_link"/>
     <axis xyz="0 0 1"/>
-    <limit upper="0.95" lower="-0.83" velocity="1" effort="100"/>
+    <limit upper="0.99" lower="-0.83" velocity="1" effort="100"/>
   </joint>
 <joint name="riel1_joint" type="fixed">
@@ -109,5 +109,5 @@
     <child link="carrier_link"/>
     <axis xyz="1 0 0"/>
-    <limit upper="1.575" lower="-1.575" velocity="1" effort="100"/>
+    <limit upper="1.64" lower="-1.575" velocity="1" effort="100"/>
   </joint>
   <transmission name="t1">

Commit message: Adjusted limits

File: dsrbot_description/urdf/DSRbot_URDF.xacro (robot description, xacro)
@@ -109,5 +109,5 @@
     <child link="carrier_link"/>
     <axis xyz="1 0 0"/>
-    <limit upper="1.64" lower="-1.575" velocity="1" effort="100"/>
+    <limit upper="1.61" lower="-1.575" velocity="1" effort="100"/>
   </joint>
   <transmission name="t1">
